File: CarPCB/ENEL300/ENEL300.kicad_sch (KiCad schematic)
At the start: 83 parts, among them J1 Microsemi_FlashPro-JTAG-10, J2 Conn_ARM_JTAG_SWD_10, J3 USB_C_Receptacle, J4 Encoder1, J5 Encoder2, M1 Motor_DC, M2 Motor_DC, Q1 2N3904, Q2 2N3904, Q3 2N7002E, Q4 2N7002E, Q5 2N7002E, Q6 2N7002E, U1 LM2596S-5, U2 ESP32-C3-WROOM-02, U3 CH340C, U4 STM32F446RETx, U5 BQ297xy, U6 VNH5019A-E, U7 VNH5019A-E, Y1 ASE-xxxMHz, Y2 ASE-xxxMHz

Commit message: Add files via upload
Parts:
- added J6: Speaker Terminal, TerminalBlock_Phoenix:TerminalBlock_Phoenix_MPT-0,5-4-2.54_1x04_P2.54mm_Horizontal, symbol Connector:Screw_Terminal_01x04
- added J7: LED Terminal, TerminalBlock_Phoenix:TerminalBlock_Phoenix_MPT-0,5-2-2.54_1x02_P2.54mm_Horizontal, symbol Connector:Screw_Terminal_01x02
- added J8: Ultrasonic Sensor, TerminalBlock_Phoenix:TerminalBlock_Phoenix_MPT-0,5-4-2.54_1x04_P2.54mm_Horizontal, symbol Connector:Screw_Terminal_01x04
- added Q7: 2N7002E, Package_TO_SOT_SMD:SOT-23, symbol Transistor_FET:2N7002E
- added R15, R34: 220, Resistor_SMD:R_0805_2012Metric, symbol Device:R_US
- added R25: 22, Resistor_SMD:R_0805_2012Metric, symbol Device:R_US
- added R33, R35: 10k, Resistor_SMD:R_0805_2012Metric, symbol Device:R_US
- C1, C10, C11, C12, C13, C14, C15, C16, C17, C18, C19, C2, C20, C21, C22, C23, C24, C3, C4, C5, C6, C7, C8, C9: footprint (none) -> Capacitor_SMD:C_0805_2012Metric
- F1: footprint (none) -> Fuse:Fuse_1206_3216Metric
- FB1, L1: footprint (none) -> Inductor_SMD:L_0805_2012Metric
- J1: footprint (none) -> Connector_IDC:IDC-Header_2x05_P2.54mm_Vertical
- J2: footprint (none) -> Connector_PinHeader_1.27mm:PinHeader_2x05_P1.27mm_Vertical
- J3: footprint (none) -> Connector_USB:USB_C_Receptacle_GCT_USB4135-GF-A_6P_TopMnt_Horizontal
- J4, J5: footprint (none) -> Connector_FFC-FPC:Amphenol_F32Q-1A7x1-11004_1x04-1MP_P0.5mm_Horizontal
- M1, M2: footprint (none) -> TerminalBlock_Phoenix:TerminalBlock_Phoenix_MPT-0,5-2-2.54_1x02_P2.54mm_Horizontal
- R1, R10, R11, R12, R13, R14, R16, R17, R18, R19, R2, R20, R21, R22, R23, R24, R26, R27, R28, R29, R3, R30, R31, R32, R4, R5, R6, R7, R8, R9: footprint (none) -> Resistor_SMD:R_0805_2012Metric
Connections:
- net +3.3V: now also R33.1; no longer J4.1 (Pin_1), J5.1 (Pin_1)
- net GND: now also J6.4 (Pin_4), J8.4 (Pin_4), Q7.2 (S), R35.2
- net at U4.34 (PB13): now also R34.1
- net at U4.35 (PB14): now also R15.1
- net at U4.36 (PB15): now also J6.3 (Pin_3), R33.2
- net at U4.61 (PB8): now also J8.2 (Pin_2)
- net at U4.62 (PB9): now also J8.3 (Pin_3)
- new net: Q7.1 (G), R34.2, R35.1
- new net: Q7.3 (D), R25.1
- new net: J7.2 (Pin_2), R25.2
- new net: J6.2 (Pin_2), R15.2
- new net +5V: J4.1 (Pin_1), J5.1 (Pin_1), J6.1 (Pin_1), J7.1 (Pin_1), J8.1 (Pin_1)
Other:
- moved on the sheet: J4, J5
